File: Pneumatics Card/pneu_pwr_brd_11_19_25.kicad_sch (KiCad schematic)
At the start: 62 parts, among them J1 2X1, J10 Conn_01x02, J11 Conn_01x02, J12 2X1, J2 2X1, J3 2X1, J4 2X1, J5 2X1, J6 2X1, J7 Conn_01x03_Pin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

Commit message: a
Parts:
- C1: value 10nF -> 22nF
- C12: value 4.7u -> 0.47u
- R1: value 100k -> 1k
- R2: value 150k -> 3.9k
Changed lines of the file:
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@@
 			)
 		)
-		(property "Value" "10nF"
+		(property "Value" "22nF"
 			(at 69.342 124.968 0)
 			(effects
@@
 			)
 		)
-		(property "Value" "150k"
+		(property "Value" "3.9k"
 			(at 52.07 139.7 0)
 			(effects
@@
 			)
 		)
-		(property "Value" "4.7u"
+		(property "Value" "0.47u"
 			(at 90.17 124.46 0)
 			(effects
@@
 			)
 		)
-		(property "Value" "100k"
+		(property "Value" "1k"
 			(at 52.07 129.54 0)
 			(effects
