File: Pneumatics Card/pneu_pwr_brd_11_19_25.kicad_pcb (KiCad board)
At the start: 4 copper layers, 65 x 65 mm, 79 parts, among them J1 2X1, J10 Conn_01x02, J11 Conn_01x02, J12 2X1, J13 2X1, J2 2X1, J3 2X1, J4 2X1, J5 2X1, J6 2X1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

Commit message: Changed some Silk-screen and measured hole size
Other:
- board text added: "3.3V GND GND"
- board text added: "NRST SWDIO SWCLK"
Changed lines of the file:
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@@
 		(tags "Through hole pin header THT 1x03 2.54mm single row")
 		(property "Reference" "J7"
-			(at 2.6975 3.1375 0)
+			(at -0.03 -3.03 0)
 			(layer "F.SilkS")
 			(effects
@@
 	)
 	(gr_text "USART_TX"
-		(at 122.23 81.11 90)
+		(at 122.23 81.06 90)
 		(layer "F.SilkS")
 		(effects
 			(font
 				(size 0.5 0.5)
-				(thickness 0.075)
+				(thickness 0.125)
+				(bold yes)
 			)
 			(justify left bottom)
@@
 		)
 	)
+	(gr_text "3.3V GND GND"
+		(at 138.02 61.23 90)
+		(layer "F.SilkS")
+		(effects
+			(font
+				(size 0.5 0.5)
+				(thickness 0.125)
+			)
+			(justify left bottom)
+		)
+	)
 	(gr_text "GND"
 		(at 103.85 81.61 90)
@@
 		)
 	)
+	(gr_text "NRST SWDIO SWCLK\n"
+		(at 127.04 73.49 0)
+		(layer "F.SilkS")
+		(effects
+			(font
+				(size 0.5 0.5)
+				(thickness 0.125)
+			)
+			(justify left bottom)
+		)
+	)
 	(gr_text "Fuse"
 		(at 95.17 74.14 0)
@@
 			(font
 				(size 0.5 0.5)
-				(thickness 0.075)
+				(thickness 0.125)
+				(bold yes)
 			)
 			(justify left bottom)
