File: Pneumatics Card/pneumatics_card_10-22-25-PCA/pneumatics_card_10-22-25/pneu_pwr_brd.kicad_sch (KiCad schematic)
At the start: 57 parts, among them J2 2X1, J3 2X1, J4 2X1, J5 2X1, J6 2X1, J7 2X1, Q3 FQP30N06L, Q4 FQP30N06L, Q5 FQP30N06L, Q6 FQP30N06L, Q7 IRF4905SPbF, U1 L7805, U2 LD1117V33, U3 PCA9685, U4 MCP1416, U5 TCA4307, U6 MCP1416, U7 MCP1416, U8 MCP1416

Commit message: annotating schematic
Parts:
- renumbered C6 to C16, R14 to R20
Changed lines of the file:
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@@
 		(on_board yes)
 		(dnp no)
-		(property "Reference" "R14"
+		(property "Reference" "R20"
 			(at 66.04 30.48 0)
 			(effects
@@
 			(project "pneu_pwr_brd"
 				(path "/c299c6f2-212e-472c-8577-e7ed124513dd"
-					(reference "R14")
+					(reference "R20")
 					(unit 1)
 				)
@@
 		(on_board yes)
 		(dnp no)
-		(property "Reference" "C6"
+		(property "Reference" "C16"
 			(at 88.9 53.34 0)
 			(effects
@@
 			(project "pneu_pwr_brd"
 				(path "/c299c6f2-212e-472c-8577-e7ed124513dd"
-					(reference "C6")
+					(reference "C16")
 					(unit 1)
 				)

Commit message: old pneumatics
Parts:
- removed D5: 1N47xxA, Diode_THT:D_DO-41_SOD81_P10.16mm_Horizontal, symbol Diode:1N47xxA
- removed Q7: IRF4905SPbF, Package_TO_SOT_THT:TO-220-3_Vertical, symbol Transistor_FET:IRLZ34N
- removed R12, R13: 100k, Resistor_SMD:R_0805_2012Metric_Pad1.20x1.40mm_HandSolder, symbol PowerboardRev5-eagle-import:R-US_R0805
- added C12: 0.47u, Capacitor_SMD:C_0402_1005Metric, symbol Device:C
- added Q1: NTR0202PLT1G OR Si2347DS, Package_TO_SOT_SMD:SOT-23-3, symbol Simulation_SPICE:PMOS
- added R1: 1k, Resistor_SMD:R_0402_1005Metric, symbol PowerboardRev5-eagle-import:R-US_R0805
- added R2: 4.7k, Resistor_SMD:R_0402_1005Metric, symbol PowerboardRev5-eagle-import:R-US_R0805
- C5: value 1u -> 22nF; footprint Capacitor_THT:CP_Radial_D5.0mm_P2.00mm -> Capacitor_SMD:C_0402_1005Metric
- renumbered C14 to C13, C13 to C14, C11 to C15, C12 to C16, C7 to C17, C8 to C18, C9 to C19, C10 to C20, C6 to C25, J7 to J1, R20 to R12, R155 to R15, U3 to U10, U4 to U3, U6 to U4, U7 to U8, U8 to U9
Connections:
- net 12V: now also C12.2, Q1.1 (D)
- net GND: now also R2.1; no longer C5.1
- net at F1.2: now also C5.2, Q1.3 (S), R1.2
- net +12V_fuse: now reaches F1.1, J2.1 (Pin_1)
- new net: C12.1, C5.1, Q1.2 (G), R1.1, R2.2
Other:
- moved on the sheet: J2
