File: Pneumatics Card/Nitya's Folder/pneu_pwr_brd_11_19_25.kicad_pcb (KiCad board)
At the start: 4 copper layers, 65 x 65 mm, 79 parts, among them J1 2X1, J10 Conn_01x02, J11 Conn_01x02, J12 2X1, J13 2X1, J2 2X1, J3 2X1, J4 2X1, J5 2X1, J6 2X1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

Commit message: finished back up pneumatics
Parts:
- removed BOOT_R1: 10k, Resistor_SMD:R_0805_2012Metric_Pad1.20x1.40mm_HandSolder
- removed Bulk_1: 1uF, Capacitor_SMD:C_0805_2012Metric_Pad1.18x1.45mm_HandSolder
- removed Bulk_22: 22uF, Capacitor_SMD:C_0805_2012Metric_Pad1.18x1.45mm_HandSolder
- removed Bulk_4.7: 4.7uF, Capacitor_SMD:C_0805_2012Metric_Pad1.18x1.45mm_HandSolder
- removed C10, C11: 10pF, Capacitor_SMD:C_0402_1005Metric_Pad0.74x0.62mm_HandSolder
- removed C7, C8, C9, T_Cd1, T_Cd2: 100nF, Capacitor_SMD:C_0805_2012Metric_Pad1.18x1.45mm_HandSolder
- removed J10, J11: Conn_01x02, Connector_PinHeader_2.54mm:PinHeader_1x02_P2.54mm_Vertical
- removed J12, J13: 2X1, Connector_JST:JST_PH_B2B-PH-K_1x02_P2.00mm_Vertical
- removed J7, J9: Conn_01x03_Pin, Connector_PinHeader_2.54mm:PinHeader_1x03_P2.54mm_Vertical
- removed J8: Conn_01x03, custom_components:slide_switch_EGER1218_Thruster
- removed U6: STM32G0B1RETx, Package_QFP:LQFP-64_10x10mm_P0.5mm
- removed U7: ATA6561-GAQW-N, custom_components:SOIC8_4P9X3P9MC_MCH
- removed Y1: 16Mhz, Crystal:Crystal_SMD_3225-4Pin_3.2x2.5mm
- added C30: 10u, Capacitor_THT:CP_Radial_D5.0mm_P2.00mm, F.Cu at (134.0, 58.5)
- added R3: 10k, Resistor_SMD:R_0805_2012Metric_Pad1.20x1.40mm_HandSolder, F.Cu at (127.5, 62.0)
- added U10: PCA9685, Package_SO:TSSOP-28_4.4x9.7mm_P0.65mm, F.Cu at (126.5, 54.6)
- R1: value 1k -> 4.7k
- R2: value 4.7k -> 1k
- U5: footprint custom_components:SOIC8_DGK_TEX -> TCA4307:SOP65P490X110-8N
Routing:
- net 3.3V: track 97.4 -> 40.1 mm
- net GND: track 54.1 -> 27.4 mm, vias 59 -> 51
- net (no net): track 28.2 -> 1.68 mm
- net SDA: track 10.4 -> 34.6 mm
- net SCL: track 9.23 -> 32.4 mm
- net FDCAN_RX: track 22.8 -> 0.00 mm
- net FDCAN_TX: track 20.4 -> 0.00 mm
- net /NRST: track 16.6 -> 0.00 mm
- net /SWCLK: track 14.7 -> 0.00 mm
- net /SWDIO: track 13.1 -> 0.00 mm
- net +5V: track 0.00 -> 12.5 mm
- net CAN+: track 12.4 -> 0.00 mm
- net CAN-: track 12.3 -> 0.00 mm
- net 5V: track 25.3 -> 14.2 mm, vias 2 -> 1
- net Net-(J8-Pin_2): track 7.88 -> 0.00 mm
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Other:
- board text removed: "CAN- CAN+"
- board text removed: "NRST SWDIO SWCLK"
- board text removed: "USART_RX"
- board text removed: "USART_TX"
